File: Hardware/H616_devboard.kicad_pcb (KiCad board)
At the start: 4 copper layers, 26.5 x 72.5 mm, 125 parts, among them J1 Micro_SD_Card_Det2, J2 USB_C_Receptacle_USB2.0, J3 USB_C_Receptacle_USB2.0, U1 H616, U2 DDR3 FBGA-96, U3 AXP305, U4 CP2102N-Axx-xQFN28, Y1 25MHz

Commit message: fixed crystal resonator value
Parts:
- U2: value DDR3 FBGA-96 -> K4B8G1646D
- Y1: value 25MHz -> 24MHz
