File: Hardware/dram.kicad_sch (KiCad schematic)
At the start: 22 parts, among them U1 H616, U2 DDR3 FBGA-96

Commit message: fixed crystal resonator value
Parts:
- R5: now not fitted
- U2: value DDR3 FBGA-96 -> K4B8G1646D
