File: Hardware/io1.kicad_sch (KiCad schematic)
At the start: 20 parts, among them J1 Micro_SD_Card_Det2, U1 H616

Commit message: fixed crystal resonator value
Parts:
- renumbered TP2 to TP11, TP2 to TP12, TP2 to TP13
